File: Main_Board_V1/MOSAIC Main Board.kicad_pcb (KiCad board)
At the start: 2 copper layers, 318 x 186 mm, 83 parts, among them J1 CONN E, J10 QWIIC_RIGHT_ANGLE, J11 Vertical Qwiic Connector, J12 CONN E, J13 CONN E, J14 35RAPC4BH3 CONN 3.5MM, J2 CONN E, J3 CONN E, J4 CONN HEADER VERT 10POS 1.27MM, J5 USB TYPE C R/A SMT 16PIN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

Commit message: Added ground plane to new board outline
Routing:
- net 3.3V: track 285.3 -> 0.00 mm, vias 15 -> 0
- net /I2C_~{INT}: track 256.3 -> 0.00 mm, vias 12 -> 0
- net /I2C_SCL: track 213.4 -> 0.00 mm, vias 7 -> 0
- net GND: track 199.2 -> 0.00 mm, vias 83 -> 0
- net /SPI_PROCESSOR_SDO: track 188.6 -> 0.00 mm, vias 13 -> 0
- net /SPI_PROCESSOR_SCK: track 181.2 -> 0.00 mm, vias 12 -> 0
- net /SPI_PROCESSOR_SDI: track 177.6 -> 0.00 mm, vias 13 -> 0
- net /~{RESET}: track 175.5 -> 0.00 mm, vias 12 -> 0
- net /I2C_SDA: track 161.0 -> 0.00 mm, vias 7 -> 0
- net /G4-PROCESSOR/SD_CARD_~{CS}: track 143.3 -> 0.00 mm, vias 9 -> 0
- net V_BATT: track 129.6 -> 0.00 mm, vias 4 -> 0
- net VCC: track 127.3 -> 0.00 mm, vias 6 -> 0
- net /D1-PROCESSOR: track 126.2 -> 0.00 mm, vias 3 -> 0
- net /G6-JUMPER: track 121.7 -> 0.00 mm, vias 12 -> 0
- net /TX2-PROCESSOR: track 120.1 -> 0.00 mm, vias 5 -> 0
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
Commit message: Deleted old tracks and started organizing surface components
Parts:
- moved C2 485.7 mm to (364.9, 178.3)
- moved C3 485.7 mm to (367.7, 178.3)
- moved C5 485.7 mm to (383.7, 182.7)
- moved C7 485.7 mm to (385.4, 182.7)
- moved D6 485.7 mm to (371.3, 174.7)
- moved Q1 485.7 mm to (369.5, 165.6)
- moved R10 485.7 mm to (361.4, 166.2)
- moved R13 485.7 mm to (370.7, 178.3)
- moved UNK3V3_MEAS1 485.7 mm to (340.2, 150.2)
- moved UNK5V_MEAS1 485.7 mm to (336.2, 150.1)
- moved VE1 485.7 mm to (328.6, 159.6)
- moved D4 485.7 mm to (365.0, 172.2)
- moved U4 485.7 mm to (373.8, 178.3)
- moved F1 423.2 mm to (343.5, 36.0), turned to -90 degrees
- moved BYP1 423.0 mm to (348.4, 36.0), turned to 180 degrees
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
Commit message: Wired/Placed processor/x2 module connectors
Parts:
- moved R6 212.5 mm to (100.1, 93.2), turned to -90 degrees
- moved U1 209.9 mm to (103.8, 95.2), turned to 90 degrees
- moved R5 207.1 mm to (100.1, 97.0), turned to 90 degrees
- moved BYP1 197.5 mm to (161.4, 99.5)
- moved F1 197.5 mm to (156.5, 99.5)
- moved R8 197.5 mm to (160.0, 88.5)
- moved R9 197.5 mm to (160.0, 91.0)
- moved U2 197.5 mm to (160.0, 95.0)
- moved J5 197.5 mm to (170.3, 94.8)
- moved H1 159.7 mm to (146.1, 133.4)
- moved H2 159.6 mm to (146.1, 95.2)
- moved J2 137.6 mm to (119.3, 95.9)
- moved H3 137.4 mm to (139.6, 99.9)
- moved J1 136.9 mm to (103.9, 114.3)
- moved J3 136.9 mm to (103.9, 76.1)
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Routing:
- net GND: track 0.00 -> 101.3 mm, vias 0 -> 47
- net /I2C_SDA: track 0.00 -> 98.1 mm, vias 0 -> 8
- net /I2C_SCL: track 0.00 -> 97.5 mm, vias 0 -> 7
- net /I2C_~{INT}: track 0.00 -> 85.8 mm, vias 0 -> 8
- net /~{RESET}: track 0.00 -> 85.4 mm, vias 0 -> 5
- net 3.3V: track 0.00 -> 77.7 mm, vias 0 -> 4
- net /G0-PROCESSOR: track 0.00 -> 62.0 mm, vias 0 -> 3
- net /SPI_PROCESSOR_SDI: track 0.00 -> 61.5 mm, vias 0 -> 5
- net /D1-PROCESSOR: track 0.00 -> 61.3 mm, vias 0 -> 3
- net /SDIO_DATA2/PWR_EN0_ALT: track 0.00 -> 58.6 mm, vias 0 -> 1
- net /G4-PROCESSOR/SD_CARD_~{CS}: track 0.00 -> 56.4 mm, vias 0 -> 1
- net /G3-PROCESSOR: track 0.00 -> 55.8 mm, vias 0 -> 1
- net /RX2-PROCESSOR: track 0.00 -> 55.4 mm, vias 0 -> 3
- net /G2-PROCESSOR: track 0.00 -> 55.0 mm, vias 0 -> 1
- net /G1-PROCESSOR: track 0.00 -> 54.5 mm, vias 0 -> 1
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- added copper zone on B.Cu, net 3.3V
Other:
- board size 318 x 186 mm -> 89 x 89 mm

Commit message: Lots of placements and routing
Parts:
- moved C5 258.5 mm to (142.1, 76.3), turned to 180 degrees
- moved C7 257.1 mm to (142.1, 78.0), turned to 180 degrees
- moved VIN 256.3 mm to (156.4, 107.7)
- moved U4 247.8 mm to (146.7, 79.3), turned to -90 degrees
- moved R13 242.1 mm to (149.8, 79.2), turned to 90 degrees
- moved D6 240.4 mm to (149.2, 82.8), turned to 180 degrees
- moved C3 236.6 mm to (152.8, 79.2), turned to 90 degrees
- moved Q1 232.1 mm to (149.8, 90.8), turned to 180 degrees
- moved C2 231.5 mm to (155.6, 79.2), turned to 90 degrees
- moved D4 230.6 mm to (151.0, 86.4), turned to 180 degrees
- moved R10 219.6 mm to (154.6, 92.3), turned to -90 degrees
- moved UNK3V3_MEAS1 207.3 mm to (142.3, 88.4), turned to 90 degrees
- moved J14 200.8 mm to (160.4, 83.0)
- moved UNK5V_MEAS1 200.7 mm to (145.2, 88.5), turned to 90 degrees
- moved J9 197.0 mm to (169.4, 71.3)
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- renumbered TP2 to VIN
Routing:
- net /I2C_SCL1-PROCESSOR/QWIIC_EN: track 0.00 -> 104.3 mm, vias 0 -> 8
- net /SPI_PROCESSOR_SDO: track 35.1 -> 138.5 mm, vias 3 -> 9
- net /I2C_SDA1-PROCESSOR/~{SD_ENABLE}: track 0.00 -> 100.3 mm, vias 0 -> 6
- net /SPI_PROCESSOR_SDI: track 61.5 -> 157.9 mm, vias 5 -> 11
- net /SPI_PROCESSOR_SCK: track 33.8 -> 129.1 mm, vias 3 -> 9
- net /G4-PROCESSOR/SD_CARD_~{CS}: track 56.4 -> 148.4 mm, vias 1 -> 4
- net /I2C_~{INT}: track 85.8 -> 160.1 mm, vias 8 -> 10
- net 3.3V: track 77.7 -> 151.3 mm, vias 4 -> 6
- net /D+: track 5.39 -> 59.7 mm, vias 0 -> 4
- net /D-: track 5.58 -> 59.0 mm, vias 0 -> 4
- net GND: track 101.3 -> 152.4 mm, vias 47 -> 75
- net V_BATT: track 0.00 -> 45.9 mm, vias 0 -> 2
- net V_USB: track 10.1 -> 32.6 mm, vias 0 -> 1
- net /RBF_BATT_IN: track 0.00 -> 15.3 mm
- net VIN: track 20.8 -> 35.8 mm
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
Commit message: More placement and routing work
Parts:
- moved J11 180.8 mm to (165.6, 116.6)
- moved R16 180.8 mm to (165.4, 110.2)
- moved I2C_PU1 180.8 mm to (164.1, 105.5)
- moved J10 180.8 mm to (167.7, 116.6)
- moved R15 180.8 mm to (162.5, 110.1)
- moved S5 141.0 mm to (100.0, 115.2)
- moved S4 139.3 mm to (100.0, 120.8)
- moved C6 130.5 mm to (157.4, 123.8)
- moved C8 130.5 mm to (167.8, 123.8)
- moved R14 130.5 mm to (160.3, 123.8)
- moved U5 130.5 mm to (163.8, 123.9)
- moved J6 118.5 mm to (79.4, 109.4)
- moved J7 118.5 mm to (79.4, 105.6)
- moved S2 88.7 mm to (97.4, 107.6), turned to 90 degrees
- moved S1 61.4 mm to (97.4, 80.5), turned to 90 degrees
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Routing:
- net VCC: track 3.42 -> 169.5 mm, vias 0 -> 9
- net /G6-JUMPER: track 0.00 -> 77.1 mm, vias 0 -> 8
- net /I2C_SCL: track 97.5 -> 150.5 mm, vias 7 -> 9
- net /I2C_SDA: track 98.1 -> 148.0 mm, vias 8 -> 12
- net /SDIO_DATA2/PWR_EN0_ALT: track 58.2 -> 103.4 mm, vias 1 -> 5
- net /~{CS1}-PROCESSOR: track 0.00 -> 44.6 mm, vias 0 -> 2
- net 3.3V: track 151.3 -> 193.4 mm, vias 6 -> 10
- net /G6-PROCESSOR: track 0.00 -> 37.6 mm, vias 0 -> 1
- net /I2C_SCL1-PROCESSOR/QWIIC_EN: track 104.3 -> 138.3 mm
- net /SPI_PROCESSOR_SCK: track 129.1 -> 162.8 mm, vias 9 -> 12
- net /SDIO_DATA1/PWR_EN1_ALT: track 26.8 -> 52.7 mm, vias 3 -> 7
- net /G5-JUMPER: track 0.00 -> 20.2 mm, vias 0 -> 2
- net /A1-PROCESSOR/~{CS1}-ALT: track 36.3 -> 56.0 mm, vias 3 -> 4
- net VIN: track 35.8 -> 55.1 mm, vias 0 -> 2
- net /~{BOOT}: track 47.3 -> 60.3 mm, vias 1 -> 2
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
Commit message: More placement and routing work
Parts:
- moved D1 145.3 mm to (164.0, 133.0)
- moved UNK5V_LED1 144.1 mm to (164.1, 137.0), turned to 0 degrees
- moved DIVIDER1 140.7 mm to (143.6, 115.8), turned to 90 degrees
- moved R3 136.5 mm to (164.1, 134.8), turned to 0 degrees
- moved J4 133.9 mm to (108.2, 131.5), turned to -90 degrees
- moved R1 129.5 mm to (141.1, 117.8)
- moved R2 129.5 mm to (141.1, 113.5)
- moved D2 127.4 mm to (152.4, 133.0), turned to 0 degrees
- moved R7 127.2 mm to (158.2, 134.8)
- moved R4 125.7 mm to (152.5, 134.8), turned to 0 degrees
- moved UNK3V3_LED1 125.0 mm to (152.5, 137.0), turned to 0 degrees
- moved D3 117.9 mm to (158.2, 133.0), turned to 0 degrees
- moved QWIIC_LED1 117.3 mm to (158.3, 137.0), turned to 0 degrees
- moved VE1 80.1 mm to (137.6, 86.8), turned to 90 degrees
- moved J7 35.1 mm to (103.0, 131.6)
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Routing:
- net VIN: track 55.1 -> 155.2 mm, vias 2 -> 9
- net 3.3V: track 193.4 -> 264.5 mm, vias 10 -> 14
- net /VIN/3: track 0.00 -> 49.5 mm, vias 0 -> 4
- net /SWDIO: track 0.00 -> 38.7 mm, vias 0 -> 3
- net /3.3V_EN: track 0.00 -> 29.4 mm, vias 0 -> 4
- net /~{RESET}: track 94.1 -> 115.2 mm
- net 3.3V_QWIIC: track 12.7 -> 27.7 mm
- net Net-(U4-EN): track 4.84 -> 19.2 mm, vias 0 -> 2
- net Net-(D1-PadC): track 0.00 -> 4.58 mm
- net Net-(D2-PadC): track 0.00 -> 4.57 mm
- net Net-(D3-PadC): track 0.00 -> 4.56 mm
- net Net-(DIVIDER1-Pad2): track 0.00 -> 4.43 mm
- net Net-(D2-PadA): track 0.00 -> 1.84 mm
- net Net-(D1-PadA): track 0.00 -> 1.84 mm
- net Net-(D3-PadA): track 0.00 -> 1.82 mm
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Other:
- board text added: "3.3V Power"
- board text added: "5V Power"
- board text added: "QWIIC Power"

Commit message: More placement and routing
Parts:
- added GND: ~, main_board_footprints_V1.0:1X01_NO_SILK, F.Cu at (169.8, 111.3)
- moved SWDIO 310.2 mm to (169.8, 107.7)
- moved 3.3V 270.9 mm to (169.8, 104.1)
- moved V_BATT 247.7 mm to (169.8, 109.5)
- moved VIN 12.6 mm to (169.8, 105.9)
- moved D5 12.6 mm to (166.6, 65.4)
- moved R4 2.70 mm to (155.2, 134.8)
- moved UNK3V3_LED1 2.70 mm to (155.2, 137.0)
- moved D2 2.70 mm to (155.1, 133.0)
- moved D3 1.38 mm to (159.6, 133.0)
- moved R7 1.38 mm to (159.6, 134.8)
- moved QWIIC_LED1 1.38 mm to (159.7, 137.0)
- moved S1 0.62 mm to (96.8, 80.5)
- moved S2 0.62 mm to (96.8, 107.6)
- moved S3 0.62 mm to (96.8, 70.1)
- renumbered TP3 to 3.3V, TP4 to SWDIO, TP1 to V_BATT
Connections:
- S1 pad GND1: (no net) -> GND
- S1 pad GND2: (no net) -> GND
- S1 pad GND3: (no net) -> GND
- S1 pad GND4: (no net) -> GND
- S2 pad GND1: (no net) -> GND
- S2 pad GND2: (no net) -> GND
- S2 pad GND3: (no net) -> GND
- S2 pad GND4: (no net) -> GND
- S3 pad GND1: (no net) -> GND
- S3 pad GND2: (no net) -> GND
- S3 pad GND3: (no net) -> GND
- S3 pad GND4: (no net) -> GND
Routing:
- net GND: track 153.0 -> 236.8 mm, vias 75 -> 110
- net /SWDIO: track 38.7 -> 109.9 mm, vias 3 -> 5
- net 3.3V: track 264.5 -> 315.6 mm, vias 14 -> 19
- net /SWDCK: track 0.00 -> 41.0 mm, vias 0 -> 2
- net V_BATT: track 45.9 -> 74.5 mm, vias 2 -> 4
- net /RBF_USB_IN: track 6.99 -> 26.5 mm, vias 0 -> 1
- net /SPI_PROCESSOR_SDO: track 138.4 -> 153.9 mm, vias 9 -> 11
- net Net-(U3-STAT): track 3.19 -> 17.2 mm, vias 0 -> 2
- net VIN: track 155.2 -> 165.1 mm, vias 9 -> 10
- net Net-(D5-PadA): track 10.8 -> 17.9 mm
- net /SPI_PROCESSOR_SDI: track 157.9 -> 161.8 mm
- net /G7-PROCESSOR: track 28.0 -> 31.8 mm
- net /PWM1-PROCESSOR: track 31.1 -> 33.8 mm
- net /D-: track 60.0 -> 62.7 mm
- net /D+: track 60.3 -> 62.8 mm
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Other:
- board text added: "Test Points"
- board text removed: "3.3V QWIIC"

Commit message: More placement and routing
Parts:
- removed the GND at (169.8, 111.3)
- added G***: LOGO, LOGO, F.Cu at (117.0, 132.4)
- added GND: ~, main_board_footprints_V1.0:PAD.03X.05, F.Cu at (169.7, 106.1)
- H3: moved to F.Cu
- H4: moved to B.Cu
- moved LOGO1 258.7 mm to (159.2, 116.3)
- moved VIN 3.42 mm to (169.7, 109.3)
- moved V_BATT 1.42 mm to (169.7, 110.9)
- moved 3.3V 0.43 mm to (169.7, 104.5)
- moved SWDIO 0.10 mm to (169.7, 107.7)
- turned H4 to -90 degrees
Connections:
- S1 pad GND1: GND -> (no net)
- S1 pad GND2: GND -> (no net)
- S1 pad GND3: GND -> (no net)
- S1 pad GND4: GND -> (no net)
- S2 pad GND1: GND -> (no net)
- S2 pad GND2: GND -> (no net)
- S2 pad GND3: GND -> (no net)
- S2 pad GND4: GND -> (no net)
- S3 pad GND1: GND -> (no net)
- S3 pad GND2: GND -> (no net)
- S3 pad GND3: GND -> (no net)
- S3 pad GND4: GND -> (no net)
Routing:
- net /SWDIO: track 109.9 -> 104.1 mm
- net VIN: track 165.1 -> 161.7 mm
- net V_BATT: track 74.5 -> 76.4 mm
- net /SPI_SCK1-PROCESSOR: track 30.6 -> 32.3 mm
- net /I2C_~{INT}: track 160.2 -> 160.9 mm
- net /I2C_SCL: track 152.0 -> 152.5 mm
- net GND: vias 110 -> 113
Other:
- board text added: "3.3V MEAS"
- board text added: "5V MEAS"
- board text added: "Function Board"
- board text added: "MOSAIC"
- board text added: "Main Board"
- board text removed: "MOSAIC MAIN BOARD"
