File: Main_Board_V1/MOSAIC Main Board.kicad_sch (KiCad schematic)
At the start: 81 parts, among them J1 CONN E, J10 QWIIC_RIGHT_ANGLE, J11 Vertical Qwiic Connector, J12 CONN E, J13 CONN E, J14 35RAPC4BH3 CONN 3.5MM, J2 CONN E, J3 CONN E, J4 CONN HEADER VERT 10POS 1.27MM, J5 USB TYPE C R/A SMT 16PIN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

Commit message: More placement and routing
Parts:
- added SWDIO1: ~, main_board_footprints_V1.0:PAD.03X.05, symbol main_board_symbols_V1.0:TEST-POINT3X5
- renumbered TP3 to 3.3V, TP4 to SWDIO, TP2 to VIN, TP1 to V_BATT
Connections:
- net GND: now also SWDIO1.1
Changed lines of the file:
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@@
 	(wire
 		(pts
-			(xy 271.018 155.448) (xy 268.478 155.448)
+			(xy 270.9406 154.5376) (xy 268.4006 154.5376)
 		)
 		(stroke
@@
 		)
 	)
+	(wire
+		(pts
+			(xy 268.4646 160.5027) (xy 271.0046 160.5027)
+		)
+		(stroke
+			(width 0.1524)
+			(type solid)
+		)
+	)
 	(polyline
 		(pts
@@
 	)
 	(label "SWDIO"
-		(at 268.478 155.448 180)
+		(at 268.4006 154.5376 180)
 		(effects
 			(font
@@
 	(symbol
 		(lib_id "main_board_symbols_V1.0:TEST-POINT3X5")
-		(at 271.018 155.448 0)
+		(at 270.9406 154.5376 0)
 		(unit 1)
 		(exclude_from_sim no)
@@
 		(on_board yes)
 		(dnp no)
-		(property "Reference" "TP4"
-			(at 276.098 155.448 0)
+		(property "Reference" "SWDIO"
+			(at 276.0206 154.5376 0)
 			(effects
 				(font
@@
 		)
 		(property "Value" "~"
-			(at 268.478 157.988 0)
+			(at 268.4006 157.0776 0)
 			(effects
 				(font
@@
 		)
 		(property "Footprint" "main_board_footprints_V1.0:PAD.03X.05"
-			(at 271.018 155.448 0)
+			(at 270.9406 154.5376 0)
 			(effects
 				(font
@@
 		)
 		(property "Datasheet" ""
-			(at 271.018 155.448 0)
+			(at 270.9406 154.5376 0)
 			(effects
 				(font
@@
 		)
 		(property "Description" ""
-			(at 271.018 155.448 0)
+			(at 270.9406 154.5376 0)
 			(effects
 				(font
@@
 			(project "MOSAIC Main Board"
 				(path "/52f21295-3640-410f-ad83-534235adfded"
-					(reference "TP4")
+					(reference "SWDIO")
 					(unit 1)
 				)
@@
 		(on_board yes)
 		(dnp no)
-		(property "Reference" "TP3"
+		(property "Reference" "3.3V"
 			(at 273.558 147.828 0)
 			(effects
@@
 			(project "MOSAIC Main Board"
 				(path "/52f21295-3640-410f-ad83-534235adfded"
-					(reference "TP3")
+					(reference "3.3V")
 					(unit 1)
 				)
@@
 		(on_board yes)
 		(dnp no)
-		(property "Reference" "TP1"
+		(property "Reference" "V_BATT"
 			(at 273.558 124.968 0)
 			(effects
@@
 			(project "MOSAIC Main Board"
 				(path "/52f21295-3640-410f-ad83-534235adfded"
-					(reference "TP1")
+					(reference "V_BATT")
 					(unit 1)
 				)
@@
 	(symbol
 		(lib_id "main_board_symbols_V1.0:GND")
+		(at 265.9246 160.5027 270)
+		(unit 1)
+		(exclude_from_sim no)
+		(in_bom yes)
+		(on_board yes)
+		(dnp no)
+		(fields_autoplaced yes)
+		(property "Reference" "#GND045"
+			(at 265.9246 160.5027 0)
+			(effects
+				(font
+					(size 1.27 1.27)
+				)
+				(hide yes)
+			)
+		)
+		(property "Value" "GND"
+			(at 264.6546 160.5026 90)
+			(effects
+				(font
+					(size 1.778 1.778)
+				)
+				(justify right)
+			)
+		)
+		(property "Footprint" ""
+			(at 265.9246 160.5027 0)
+			(effects
+				(font
+					(size 1.27 1.27)
+				)
+				(hide yes)
+			)
+		)
+		(property "Datasheet" ""
+			(at 265.9246 160.5027 0)
+			(effects
+				(font
+					(size 1.27 1.27)
+				)
+				(hide yes)
+			)
+		)
+		(property "Description" ""
+			(at 265.9246 160.5027 0)
+			(effects
+				(font
+					(size 1.27 1.27)
+				)
+				(hide yes)
+			)
+		)
+		(pin "1"
+		)
+		(instances
+			(project ""
+				(path "/52f21295-3640-410f-ad83-534235adfded"
+					(reference "#GND045")
+					(unit 1)
+				)
+			)
+		)
+	)
+	(symbol
+		(lib_id "main_board_symbols_V1.0:GND")
 		(at 367.665 139.7 0)
 		(mirror y)
@@
 		(on_board yes)
 		(dnp no)
-		(property "Reference" "TP2"
+		(property "Reference" "VIN"
 			(at 273.558 135.128 0)
 			(effects
@@
 			(project "MOSAIC Main Board"
 				(path "/52f21295-3640-410f-ad83-534235adfded"
-					(reference "TP2")
+					(reference "VIN")
 					(unit 1)
 				)
@@
 					(unit 1)
 				)
+			)
+		)
+	)
+	(symbol
+		(lib_id "main_board_symbols_V1.0:TEST-POINT3X5")
+		(at 271.0046 160.5027 0)
+		(unit 1)
+		(exclude_from_sim no)
+		(in_bom yes)
+		(on_board yes)
+		(dnp no)
+		(property "Reference" "SWDIO1"
+			(at 276.0846 160.5027 0)
+			(effects
+				(font
+					(size 1.778 1.778)
+				)
+				(justify left bottom)
+				(hide yes)
+			)
+		)
+		(property "Value" "~"
+			(at 268.4646 163.0427 0)
+			(effects
+				(font
+					(size 1.778 1.778)
+				)
+				(justify left bottom)
+				(hide yes)
+			)
+		)
+		(property "Footprint" "main_board_footprints_V1.0:PAD.03X.05"
+			(at 271.0046 160.5027 0)
+			(effects
+				(font
+					(size 1.27 1.27)
+				)
+				(hide yes)
+			)
+		)
+		(property "Datasheet" ""
+			(at 271.0046 160.5027 0)
+			(effects
+				(font
+					(size 1.27 1.27)
+				)
+				(hide yes)
+			)
+		)
+		(property "Description" ""
+			(at 271.0046 160.5027 0)
+			(effects
+				(font
+					(size 1.27 1.27)
+				)
+			)
+		)
+		(pin "1"
+		)
+		(instances
+			(project "MOSAIC Main Board"
+				(path "/52f21295-3640-410f-ad83-534235adfded"
+					(reference "SWDIO1")
+					(unit 1)
+				)

Commit message: Placement and routing
Parts:
- renumbered 3.3V to 3.3V1, SWDIO1 to GND1, SWDIO to SWDIO2, VIN to VIN1, V_BATT to V_BATT1
Changed lines of the file:
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@@
 		(on_board yes)
 		(dnp no)
-		(property "Reference" "SWDIO"
+		(property "Reference" "SWDIO2"
 			(at 276.0206 154.5376 0)
 			(effects
@@
 			(project "MOSAIC Main Board"
 				(path "/52f21295-3640-410f-ad83-534235adfded"
-					(reference "SWDIO")
+					(reference "SWDIO2")
 					(unit 1)
 				)
@@
 		(on_board yes)
 		(dnp no)
-		(property "Reference" "3.3V"
+		(property "Reference" "3.3V1"
 			(at 273.558 147.828 0)
 			(effects
@@
 			(project "MOSAIC Main Board"
 				(path "/52f21295-3640-410f-ad83-534235adfded"
-					(reference "3.3V")
+					(reference "3.3V1")
 					(unit 1)
 				)
@@
 		(on_board yes)
 		(dnp no)
-		(property "Reference" "V_BATT"
+		(property "Reference" "V_BATT1"
 			(at 273.558 124.968 0)
 			(effects
@@
 			(project "MOSAIC Main Board"
 				(path "/52f21295-3640-410f-ad83-534235adfded"
-					(reference "V_BATT")
+					(reference "V_BATT1")
 					(unit 1)
 				)
@@
 		(on_board yes)
 		(dnp no)
-		(property "Reference" "VIN"
+		(property "Reference" "VIN1"
 			(at 273.558 135.128 0)
 			(effects
@@
 			(project "MOSAIC Main Board"
 				(path "/52f21295-3640-410f-ad83-534235adfded"
-					(reference "VIN")
+					(reference "VIN1")
 					(unit 1)
 				)
@@
 		(on_board yes)
 		(dnp no)
-		(property "Reference" "SWDIO1"
+		(property "Reference" "GND1"
 			(at 276.0846 160.5027 0)
 			(effects
@@
 			(project "MOSAIC Main Board"
 				(path "/52f21295-3640-410f-ad83-534235adfded"
-					(reference "SWDIO1")
+					(reference "GND1")
 					(unit 1)
 				)

Commit message: Updating JLCPCB sources
Parts:
- BYP1, DIVIDER1, J4: now left out of the parts list
- F1: JLCPCB Part # (none) -> C135353; Source https://www.digikey.com/en/products/detail/littelfuse-inc/1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 -> (none)
- J1, J12, J13, J2, J3: JLCPCB Part # (none) -> C2977809; Source https://www.digikey.com/en/products/detail/te-connectivity-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 -> (none)
- J10: JLCPCB Part # (none) -> C295747; Source https://www.sparkfun.com/products/14417 -> (none)
- J5: JLCPCB Part # (none) -> C5409177; Source https://www.digikey.com/en/products/detail/amphenol-cs-fci/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 -> (none)
- Q1: JLCPCB Part # (none) -> C144996; Source https://www.digikey.com/en/products/detail/vishay-siliconix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 -> (none)
- R1: value 20k -> 19.6k; symbol main_board_symbols_V1.0:20KOHM-0603-1/10W-1% -> main_board_symbols_V1.0:19.6KOHM-0603-1/10W-1%; JLCPCB Part # (none) -> C22898; Source https://www.digikey.com/en/products/detail/panasonic-electr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 -> (none)
- R10: JLCPCB Part # (none) -> C840630
- R2: JLCPCB Part # (none) -> C840630; Source https://www.digikey.com/en/products/detail/bourns-inc/CR060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 -> (none)
- R8, R9: JLCPCB Part # (none) -> C14677; Source https://www.digikey.com/en/products/detail/yageo/RC0603JR-0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 -> (none)
- S1, S2, S3: JLCPCB Part # (none) -> C19188866; Source https://www.sparkfun.com/products/10860 -> (none)
- U2: JLCPCB Part # (none) -> C531179; Source https://www.mouser.com/ProductDetail/Diodes-Incorporated/D5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 -> (none)
